File: pcb/microm_schem2.brd (EAGLE design)
At the start: 101.6 x 81.3 mm, 88 parts, among them Q1 16 MHz

Commit message: Fix LED resistors.
Parts:
- 3.3V, 5V, 7.4V: value green, 2mA, 3V -> green, 2mA, 2.2V
- BT_CON: value blue, 2mA, 3V -> blue, 2mA, 2.2V
- C18, C19, C20: value 10 uF -> 10uF
- LED1, LED2, LED3, LED4, LED5: value red, 2mA, 2.1V -> red, 2mA, 1.5V
- R2: value 1.2kΩ -> 1.5kΩ
- R3, R9: value 180Ω -> 560Ω
- R4, R5, R6, R7, R8: value 680Ω -> 1kΩ

Commit message: Final fixes.
Routing:
- net GND: vias 10 -> 13
Changed lines of the file:
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@@
 </layers>
 <board>
-<fusionsync huburn="a.YnVzaW5lc3M6bXl0dW0yNTg1" projecturn="a.YnVzaW5lc3M6bXl0dW0yNTg1I0QyMDIzMTEwNzY5NTIxMTI1Ng" f3durn="urn:adsk.wipprod:dm.lineage:aJWIQGacTsKtezZMUrZWXg" pcbguid="" lastpulledtime="" lastsyncedchangeguid="" latestrevisionid="af00876f-52f9-44c0-b205-36ed584745fc" lastsyncedrevisionid="af00876f-52f9-44c0-b205-36ed584745fc" lastboardhashguid="83c800e7-3270-6dc3-ac82-6668c55781eb" lastpushedtime="2025-02-11T01:21:41Z" linktopcb3d="true"/>
+<fusionsync huburn="a.YnVzaW5lc3M6bXl0dW0yNTg1" projecturn="a.YnVzaW5lc3M6bXl0dW0yNTg1I0QyMDIzMTEwNzY5NTIxMTI1Ng" f3durn="urn:adsk.wipprod:dm.lineage:aJWIQGacTsKtezZMUrZWXg" pcbguid="" lastpulledtime="" lastsyncedchangeguid="" latestrevisionid="c894099e-078a-4ed3-8db6-678512aa80dc" lastsyncedrevisionid="c894099e-078a-4ed3-8db6-678512aa80dc" lastboardhashguid="c82f2e2b-3fb2-1e0e-3195-725e4d28989e" lastpushedtime="2025-02-12T01:11:53Z" linktopcb3d="false"/>
 <plain>
 <dimension x1="0" y1="0" x2="101.6" y2="0" x3="50.8" y3="-10.16" textsize="1.778" layer="47"/>
@@
 <via x="12.192" y="32.131" extent="1-16" drill="0.35"/>
 <via x="74.422" y="57.404" extent="1-16" drill="0.35"/>
-<contactref element="OLED" pad="1"/>
-<contactref element="C24" pad="2"/>
 <wire x1="10.16" y1="52.07" x2="11.43" y2="52.07" width="0.75" layer="1"/>
 <wire x1="10.16" y1="22.86" x2="11.43" y2="22.86" width="0.75" layer="1"/>
@@
 <via x="38.735" y="17.145" extent="1-16" drill="0.35"/>
 <contactref element="C25" pad="2"/>
+<via x="31.28545625" y="33.64956875" extent="1-16" drill="0.3"/>
+<via x="19.05" y="45.72" extent="1-16" drill="0.35"/>
+<via x="3.429" y="39.37" extent="1-16" drill="0.35"/>
+<contactref element="OLED" pad="1"/>
+<contactref element="C24" pad="2"/>
 </signal>
 <signal name="OSC1">
@@
 <contactref element="C16" pad="1"/>
 <contactref element="μC" pad="30"/>
-<wire x1="32.08" y1="34.84" x2="32.08" y2="32.715" width="0.5" layer="1"/>
-<wire x1="32.08" y1="32.715" x2="31.623" y2="32.258" width="0.5" layer="1"/>
-<wire x1="31.623" y1="32.258" x2="31.623" y2="29.718" width="0.5" layer="1"/>
+<wire x1="32.08" y1="34.84" x2="32.08" y2="32.334" width="0.5" layer="1"/>
+<wire x1="32.08" y1="32.334" x2="31.623" y2="31.877" width="0.5" layer="1"/>
+<wire x1="31.623" y1="31.877" x2="31.623" y2="29.718" width="0.5" layer="1"/>
 <wire x1="31.623" y1="29.718" x2="31.115" y2="29.21" width="0.5" layer="1"/>
 <wire x1="31.115" y1="29.21" x2="30.419" y2="28.514" width="0.5" layer="1"/>
@@
 <wire x1="39.116" y1="42.418" x2="38.138" y2="41.44" width="0.508" layer="1"/>
 <wire x1="39.116" y1="42.418" x2="39.751" y2="42.418" width="0.508" layer="1"/>
-<wire x1="30.48" y1="34.84" x2="30.48" y2="33.147" width="0.508" layer="1"/>
-<via x="30.48" y="33.147" extent="1-16" drill="0.35"/>
+<wire x1="30.48" y1="34.84" x2="30.48" y2="33.02" width="0.508" layer="1"/>
+<via x="30.48" y="33.02" extent="1-16" drill="0.35"/>
 <wire x1="39.751" y1="40.701" x2="39.751" y2="42.418" width="1" layer="16"/>
 <wire x1="27.62" y1="32.766" x2="27.62" y2="31.369" width="1" layer="16"/>
-<wire x1="27.62" y1="32.766" x2="28.001" y2="33.147" width="1" layer="16"/>
-<wire x1="30.48" y1="33.147" x2="28.001" y2="33.147" width="1" layer="16"/>
+<wire x1="27.62" y1="32.766" x2="27.874" y2="33.02" width="1" layer="16"/>
+<wire x1="30.48" y1="33.02" x2="27.874" y2="33.02" width="1" layer="16"/>
 <wire x1="10.27039375" y1="43.815" x2="10.27039375" y2="34.65439375" width="1" layer="16"/>
 <wire x1="10.27039375" y1="34.65439375" x2="8.509" y2="32.893" width="1" layer="16"/>
