File: pcb/microm_schem2.sch (EAGLE design)
At the start: 88 parts, among them Q1 16 MHz

Commit message: Final fixes.
Changed lines of the file:
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@@
 </segment>
 <segment>
-<pinref part="GND19" gate="1" pin="GND"/>
 <pinref part="OLED" gate="A" pin="1"/>
-<wire x1="218.44" y1="147.32" x2="218.44" y2="142.24" width="0.1524" layer="91"/>
 <pinref part="C24" gate="G$1" pin="2"/>
+<wire x1="215.9" y1="142.24" x2="218.44" y2="142.24" width="0.1524" layer="91"/>
 <wire x1="218.44" y1="142.24" x2="223.52" y2="142.24" width="0.1524" layer="91"/>
 <wire x1="215.9" y1="144.78" x2="215.9" y2="142.24" width="0.1524" layer="91"/>
-<wire x1="215.9" y1="142.24" x2="218.44" y2="142.24" width="0.1524" layer="91"/>
+<pinref part="GND19" gate="1" pin="GND"/>
+<wire x1="218.44" y1="147.32" x2="218.44" y2="142.24" width="0.1524" layer="91"/>
+<junction x="218.44" y="142.24"/>
 </segment>
 </net>
